File: hw/qc_attiny/qc_attiny.kicad_pcb (KiCad board)
At the start: 2 copper layers, 50 x 35 mm, 24 parts, among them J1 USB_A, J2 AVR-ISP-6, SW1 SW_SEL, SW2 SW_RST, SW3 SW_Dec, SW4 SW_Inc, U1 ATtiny84A-SSU, U2 MIC5205-3.3YM5

Commit message: Update PCB
Parts:
- removed R12: 0R, Resistor_SMD:R_0603_1608Metric_Pad0.98x0.95mm_HandSolder
- added R1: 10k, Resistor_SMD:R_1206_3216Metric_Pad1.30x1.75mm_HandSolder, F.Cu at (126.0, 101.2)
- C2: footprint Capacitor_SMD:C_1206_3216Metric_Pad1.33x1.80mm_HandSolder -> Capacitor_Tantalum_SMD:CP_EIA-3216-18_Kemet-A_Pad1.58x1.35mm_HandSolder; moved to F.Cu
- C3: renamed from C1; moved to B.Cu
- J1: footprint Connector_USB:USB_A_Molex_67643_Horizontal -> qc_attiny:USB-A_Multicomp
- SW2: renamed from SW3; value SW_Dec -> SW_Inc
- SW3: renamed from SW4; value SW_Inc -> SW_Dec
- moved J1 9.92 mm to (107.5, 107.3), turned to 180 degrees
- moved C3 8.20 mm to (137.7, 108.5), turned to 270 degrees
- moved C2 7.84 mm to (137.6, 100.7), turned to 270 degrees
- renumbered C3 to C1, R6 to R10, R5 to R11, R7 to R2, R1 to R3, R2 to R4, R8 to R5, R3 to R6, R4 to R7, R9 to R8, R10 to R9, SW2 to SW1, SW1 to SW4, U2 to U1, U1 to U2
Connections:
- net /SEL_0 renamed /MOSI
- net /SEL_1 renamed /MISO
- net /SEL_2 renamed /SCLK
- R10 pad 2: Net-(R10-Pad2) -> +3V3
- R11 pad 1: Net-(R10-Pad2) -> +3V3
- R3 pad 1: /Dm_HIGH -> /Dp_HIGH
- R3 pad 2: /D- -> /D+
- R4 pad 1: /Dm_LOW -> /Dp_LOW
- R4 pad 2: /D- -> /D+
- R5 pad 2: /DEC -> /INC
- R6 pad 1: /Dp_HIGH -> /Dm_HIGH
- R6 pad 2: /D+ -> /D-
- R7 pad 1: /Dp_LOW -> /Dm_LOW
- R7 pad 2: /D+ -> /D-
- R8 pad 2: /INC -> /DEC
- R9 pad 2: Net-(R10-Pad2) -> +3V3
- SW2 pad 2: /DEC -> /INC
- SW3 pad 2: /INC -> /DEC
- U1 pad 3: (no net) -> Net-(R1-Pad1)
- U2 pad 10: /Dp_HIGH -> /Dm_HIGH
- U2 pad 11: /Dp_LOW -> /Dm_LOW
- U2 pad 12: /Dm_LOW -> /Dp_LOW
- U2 pad 13: /Dm_HIGH -> /Dp_HIGH
- U2 pad 2: /INC -> /DEC
- U2 pad 3: /DEC -> /INC
Routing:
- net /Vbus: track 7.35 -> 24.1 mm
- net Net-(R10-Pad2): track 8.64 -> 0.00 mm
- net /INC: track 10.6 -> 18.9 mm
- net /DEC: track 18.9 -> 10.6 mm
- net /Dp_HIGH: track 24.7 -> 20.4 mm
- net /Dm_HIGH: track 20.4 -> 24.7 mm
- net Net-(R1-Pad1): track 0.00 -> 3.98 mm
- net +3V3: track 81.5 -> 79.9 mm
- net /Dp_LOW: track 12.8 -> 11.8 mm
- net /Dm_LOW: track 11.8 -> 12.8 mm
- net /MISO: track 46.8 -> 47.7 mm
Other:
- board text added: "ATtiny QC controller Jan Vrhovec, 2021"
- board text added: "ICSP"
- board text added: "JLCJLCJLC"
- board text added: "RESET"
- board text added: "V++"
- board text added: "V--"
- board text removed: "ATtiny QC controller Jan Vrhovec, 2020"
- board text removed: "Dec"
- board text removed: "Inc"
