File: hw/qc_attiny/qc_attiny.sch (KiCad schematic (older format))
At the start: 24 parts, among them J1 USB_A, J2 AVR-ISP-6, SW1 SW_SEL, SW2 SW_RST, SW3 SW_Dec, SW4 SW_Inc, U1 ATtiny84A-SSU, U2 MIC5205-3.3YM5

Commit message: Update PCB
Parts:
- removed R12: 0R, Resistor_SMD:R_0603_1608Metric_Pad0.98x0.95mm_HandSolder, symbol Device:R
- added R1: 10k, Resistor_SMD:R_1206_3216Metric_Pad1.30x1.75mm_HandSolder, symbol Device:R
- C2: footprint Capacitor_SMD:C_1206_3216Metric_Pad1.33x1.80mm_HandSolder -> Capacitor_Tantalum_SMD:CP_EIA-3216-18_Kemet-A_Pad1.58x1.35mm_HandSolder
- J1: footprint Connector_USB:USB_A_Molex_67643_Horizontal -> qc_attiny:USB-A_Multicomp
- SW2: renamed from SW3; value SW_Dec -> SW_Inc
- SW3: renamed from SW4; value SW_Inc -> SW_Dec
- renumbered C3 to C1, C1 to C3, R6 to R10, R5 to R11, R7 to R2, R1 to R3, R2 to R4, R8 to R5, R3 to R6, R4 to R7, R9 to R8, R10 to R9, SW2 to SW1, SW1 to SW4, U2 to U1, U1 to U2
Connections:
- net labels added: MISO, MOSI, SCLK, SW1, SW2, SW3
- net labels removed: SEL_0, SEL_1, SEL_2
- wire segments 68 -> 72
Other:
- moved on the sheet: J1

Commit message: Code improvements
Parts:
- TP1: value TestPoint -> Vout+
- TP2: value TestPoint -> Vout-
Changed lines of the file:
@@
 P 10300 3200
 F 0 "TP2" V 10254 3388 50  0000 L CNN
-F 1 "TestPoint" V 10345 3388 50  0000 L CNN
+F 1 "Vout-" V 10345 3388 50  0000 L CNN
 F 2 "TestPoint:TestPoint_Pad_3.0x3.0mm" H 10500 3200 50  0001 C CNN
 F 3 "~" H 10500 3200 50  0001 C CNN
@@
 P 10300 2800
 F 0 "TP1" V 10254 2988 50  0000 L CNN
-F 1 "TestPoint" V 10345 2988 50  0000 L CNN
+F 1 "Vout+" V 10345 2988 50  0000 L CNN
 F 2 "TestPoint:TestPoint_Pad_3.0x3.0mm" H 10500 2800 50  0001 C CNN
 F 3 "~" H 10500 2800 50  0001 C CNN
